File: breeze_with_regulator/aiot_pico_pcb.kicad_pcb (KiCad board)
At the start: 4 copper layers, 90.5 x 24.7 mm, 28 parts, among them J1 Tag-Connect, U1 SHT31, U2 ITM-DYPA-B-02, U3 MAX6674, U5 DRV5032AJ

Commit message: Add files via upload
Parts:
- added R3: 10k, Resistor_SMD:R_0603_1608Metric, F.Cu at (189.8, 116.2)
- added R7: 10k, Resistor_SMD:R_0603_1608Metric, F.Cu at (185.3, 116.3)
- renumbered 3.6VRegulator to J2
Connections:
- Anemometer pad 3: /OUT -> Net-(Anemometer1-Pad3)
Routing:
- net Net-(Anemometer1-Pad3): track 0.00 -> 15.1 mm
- net /OUT: track 48.2 -> 35.3 mm
- net /SHDN: track 57.6 -> 58.1 mm
