File: breeze_without_regulator/aiot_pico_pcb-master/aiot_pico_pcb.kicad_pcb (KiCad board)
At the start: 4 copper layers, 88.9 x 28.3 mm, 25 parts, among them J1 Tag-Connect, U1 SHT31, U2 ITM-DYPA-B-02, U3 MAX6674, U5 DRV5032AJ

Commit message: Add files via upload
Parts:
- added R3: 10k, Resistor_SMD:R_0603_1608Metric, F.Cu at (151.8, 93.3)
- added R7: 10k, Resistor_SMD:R_0603_1608Metric, F.Cu at (147.8, 93.3)
- renumbered Connection to ConnectionMain1
Connections:
- ConnectionMain1 pad 2: /OUT -> Net-(ConnectionMain1-Pad2)
Routing:
- net Net-(ConnectionMain1-Pad2): track 0.00 -> 14.8 mm
- net /OUT: track 83.0 -> 69.5 mm
Changed lines of the file:
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@@
   (net 51 "Net-(J1-Pad10)")
   (net 52 "Net-(R6-Pad1)")
+  (net 53 "Net-(ConnectionMain1-Pad2)")
   (footprint "digikey-footprints:TO-92-3" (layer "F.Cu")
     (at 114.445 102 90)
@@
     (property "Sheetname" "")
     (attr through_hole)
-    (fp_text reference "Connection" (at 2.54 2.54) (layer "F.SilkS")
+    (fp_text reference "ConnectionMain1" (at 2.54 2.54) (layer "F.SilkS")
       (effects (font (size 1 1) (thickness 0.15)))
     )
@@
       (effects (font (size 1 1) (thickness 0.15)))
     )
-    (fp_text user "${REFERENCE}" (at 0 2.54) (layer "F.Fab")
+    (fp_text user "${REFERENCE}" (at 0 2.54) (layer "F.Fab") hide
       (effects (font (size 1 1) (thickness 0.15)))
     )
@@
       (net 2 "GND") (pinfunction "Pin_1") (pintype "passive"))
     (pad "2" thru_hole oval (at 0 2.54 90) (size 1.7 1.7) (drill 1) (layers *.Cu *.Mask)
-      (net 7 "/OUT") (pinfunction "Pin_2") (pintype "passive"))
+      (net 53 "Net-(ConnectionMain1-Pad2)") (pinfunction "Pin_2") (pintype "passive"))
     (pad "3" thru_hole oval (at 0 5.08 90) (size 1.7 1.7) (drill 1) (layers *.Cu *.Mask)
       (net 40 "/SHDN") (pinfunction "Pin_3") (pintype "passive"))
@@
   )
   (footprint "Resistor_SMD:R_0603_1608Metric" (layer "F.Cu")
+    (at 147.76 93.35 180)
+    (descr "Resistor SMD 0603 (1608 Metric), square (rectangular) end terminal, IPC_7351 nominal, (Body size source: IPC-SM-782 page 72, https://www.pcb-3d.com/wordpress/wp-content/uploads/ipc-sm-782a_amendment_1_and_2.pdf), generated with kicad-footprint-generator")
+    (tags "resistor")
+    (property "Sheetfile" "Fichier: aiot_pico_pcb.kicad_sch")
+    (property "Sheetname" "")
+    (attr smd)
+    (fp_text reference "R7" (at 2.1 0.07 90) (layer "F.SilkS")
+      (effects (font (size 0.8 0.8) (thickness 0.1)))
+    )
+    (fp_text value "10k" (at 0 1.43) (layer "F.Fab") hide
+      (effects (font (size 1 1) (thickness 0.15)))
+    )
+    (fp_text user "${REFERENCE}" (at 0 0) (layer "F.Fab")
+      (effects (font (size 0.4 0.4) (thickness 0.06)))
+    )
+    (fp_line (start -0.237258 0.5225) (end 0.237258 0.5225) (layer "F.SilkS") (width 0.12))
+    (fp_line (start -0.237258 -0.5225) (end 0.237258 -0.5225) (layer "F.SilkS") (width 0.12))
+    (fp_line (start -1.48 -0.73) (end 1.48 -0.73) (layer "F.CrtYd") (width 0.05))
+    (fp_line (start 1.48 -0.73) (end 1.48 0.73) (layer "F.CrtYd") (width 0.05))
+    (fp_line (start 1.48 0.73) (end -1.48 0.73) (layer "F.CrtYd") (width 0.05))
+    (fp_line (start -1.48 0.73) (end -1.48 -0.73) (layer "F.CrtYd") (width 0.05))
+    (fp_line (start 0.8 -0.4125) (end 0.8 0.4125) (layer "F.Fab") (width 0.1))
+    (fp_line (start 0.8 0.4125) (end -0.8 0.4125) (layer "F.Fab") (width 0.1))
+    (fp_line (start -0.8 -0.4125) (end 0.8 -0.4125) (layer "F.Fab") (width 0.1))
+    (fp_line (start -0.8 0.4125) (end -0.8 -0.4125) (layer "F.Fab") (width 0.1))
+    (pad "1" smd roundrect (at -0.825 0 180) (size 0.8 0.95) (layers "F.Cu" "F.Paste" "F.Mask") (roundrect_rratio 0.25)
+      (net 7 "/OUT") (pintype "passive"))
+    (pad "2" smd roundrect (at 0.825 0 180) (size 0.8 0.95) (layers "F.Cu" "F.Paste" "F.Mask") (roundrect_rratio 0.25)
+      (net 53 "Net-(ConnectionMain1-Pad2)") (pintype "passive"))
+    (model "${KICAD6_3DMODEL_DIR}/Resistor_SMD.3dshapes/R_0603_1608Metric.wrl"
+      (offset (xyz 0 0 0))
+      (scale (xyz 1 1 1))
+      (rotate (xyz 0 0 0))
+    )
+  )
+  (footprint "Resistor_SMD:R_0603_1608Metric" (layer "F.Cu")
     (at 151.4004 98.74)
     (descr "Resistor SMD 0603 (1608 Metric), square (rectangular) end terminal, IPC_7351 nominal, (Body size source: IPC-SM-782 page 72, https://www.pcb-3d.com/wordpress/wp-content/uploads/ipc-sm-782a_amendment_1_and_2.pdf), generated with kicad-footprint-generator")
@@
     (pad "4" smd rect (at 0.65 -0.25 270) (size 0.35 0.3) (layers "F.Cu" "F.Paste" "F.Mask")
       (net 36 "Net-(S2-Pad4)") (pinfunction "ON/OFF") (pintype "input"))
+  )
+  (footprint "Resistor_SMD:R_0603_1608Metric" (layer "F.Cu")
+    (at 151.77 93.35 180)
+    (descr "Resistor SMD 0603 (1608 Metric), square (rectangular) end terminal, IPC_7351 nominal, (Body size source: IPC-SM-782 page 72, https://www.pcb-3d.com/wordpress/wp-content/uploads/ipc-sm-782a_amendment_1_and_2.pdf), generated with kicad-footprint-generator")
+    (tags "resistor")
+    (property "Sheetfile" "Fichier: aiot_pico_pcb.kicad_sch")
+    (property "Sheetname" "")
+    (attr smd)
+    (fp_text reference "R3" (at 1.93 0.01 90) (layer "F.SilkS")
+      (effects (font (size 0.8 0.8) (thickness 0.1)))
+    )
+    (fp_text value "10k" (at 0 1.43) (layer "F.Fab") hide
+      (effects (font (size 1 1) (thickness 0.15)))
+    )
+    (fp_text user "${REFERENCE}" (at 0 0) (layer "F.Fab")
+      (effects (font (size 0.4 0.4) (thickness 0.06)))
+    )
+    (fp_line (start -0.237258 0.5225) (end 0.237258 0.5225) (layer "F.SilkS") (width 0.12))
+    (fp_line (start -0.237258 -0.5225) (end 0.237258 -0.5225) (layer "F.SilkS") (width 0.12))
+    (fp_line (start -1.48 0.73) (end -1.48 -0.73) (layer "F.CrtYd") (width 0.05))
+    (fp_line (start 1.48 0.73) (end -1.48 0.73) (layer "F.CrtYd") (width 0.05))
+    (fp_line (start -1.48 -0.73) (end 1.48 -0.73) (layer "F.CrtYd") (width 0.05))
+    (fp_line (start 1.48 -0.73) (end 1.48 0.73) (layer "F.CrtYd") (width 0.05))
+    (fp_line (start -0.8 0.4125) (end -0.8 -0.4125) (layer "F.Fab") (width 0.1))
+    (fp_line (start 0.8 0.4125) (end -0.8 0.4125) (layer "F.Fab") (width 0.1))
+    (fp_line (start 0.8 -0.4125) (end 0.8 0.4125) (layer "F.Fab") (width 0.1))
+    (fp_line (start -0.8 -0.4125) (end 0.8 -0.4125) (layer "F.Fab") (width 0.1))
+    (pad "1" smd roundrect (at -0.825 0 180) (size 0.8 0.95) (layers "F.Cu" "F.Paste" "F.Mask") (roundrect_rratio 0.25)
+      (net 2 "GND") (pintype "passive"))
+    (pad "2" smd roundrect (at 0.825 0 180) (size 0.8 0.95) (layers "F.Cu" "F.Paste" "F.Mask") (roundrect_rratio 0.25)
+      (net 7 "/OUT") (pintype "passive"))
+    (model "${KICAD6_3DMODEL_DIR}/Resistor_SMD.3dshapes/R_0603_1608Metric.wrl"
+      (offset (xyz 0 0 0))
+      (scale (xyz 1 1 1))
+      (rotate (xyz 0 0 0))
+    )
   )
   (footprint "Battery:BatteryHolder_Keystone_2460_1xAA" (layer "B.Cu")
@@
   (segment (start 142.8212 104.3462) (end 142.8212 98.3518) (width 0.25) (layer "F.Cu") (net 5))
   (segment (start 149.1282 98.7582) (end 150.25 99.88) (width 0.25) (layer "F.Cu") (net 5))
+  (segment (start 148.585 93.35) (end 149.62 93.35) (width 0.25) (layer "F.Cu") (net 7))
   (segment (start 198.9904 104.0096) (end 198.9904 98.1468) (width 0.25) (layer "F.Cu") (net 7))
-  (segment (start 132.92 94.83) (end 134.095 93.655) (width 0.25) (layer "F.Cu") (net 7))
+  (segment (start 151.1 91.87) (end 193.9 91.87) (width 0.25) (layer "F.Cu") (net 7))
   (segment (start 196.84 103.56) (end 197.76 104.48) (width 0.25) (layer "F.Cu") (net 7))
   (segment (start 198.52 104.48) (end 198.9904 104.0096) (width 0.25) (layer "F.Cu") (net 7))
+  (segment (start 149.62 93.35) (end 151.1 91.87) (width 0.25) (layer "F.Cu") (net 7))
   (segment (start 197.76 104.48) (end 198.52 104.48) (width 0.25) (layer "F.Cu") (net 7))
+  (segment (start 149.62 93.35) (end 150.945 93.35) (width 0.25) (layer "F.Cu") (net 7))
+  (segment (start 193.9 91.87) (end 195.685 93.655) (width 0.25) (layer "F.Cu") (net 7))
   (segment (start 196.84 102.43) (end 196.84 103.56) (width 0.25) (layer "F.Cu") (net 7))
   (segment (start 198.9904 97.3904) (end 198.9904 98.1468) (width 0.25) (layer "F.Cu") (net 7))
-  (segment (start 134.095 93.655) (end 195.685 93.655) (width 0.25) (layer "F.Cu") (net 7))
   (via (at 196.84 102.43) (size 0.8) (drill 0.4) (layers "F.Cu" "B.Cu") (net 7))
   (via (at 195.685 93.655) (size 0.8) (drill 0.4) (layers "F.Cu" "B.Cu") (net 7))
@@
   (segment (start 149.4654 97.63) (end 150.5754 98.74) (width 0.25) (layer "In2.Cu") (net 52))
   (segment (start 140.7896 99.1166) (end 143.2234 99.1166) (width 0.25) (layer "In2.Cu") (net 52))
+  (segment (start 146.745 93.16) (end 146.935 93.35) (width 0.25) (layer "F.Cu") (net 53))
+  (segment (start 132.92 94.83) (end 134.54 93.21) (width 0.25) (layer "F.Cu") (net 53))
+  (segment (start 134.54 93.16) (end 146.745 93.16) (width 0.25) (layer "F.Cu") (net 53))
+  (segment (start 134.54 93.21) (end 134.54 93.16) (width 0.25) (layer "F.Cu") (net 53))
   (zone (net 2) (net_name "GND") (layer "F.Cu") (hatch edge 0.508)
     (connect_pads (clearance 0.508))
