File: breeze_without_regulator/aiot_pico_pcb-master/aiot_pico_pcb.kicad_sch (KiCad schematic)
At the start: 25 parts, among them J1 Tag-Connect, U1 SHT31, U2 ITM-DYPA-B-02, U3 MAX6674, U5 DRV5032AJ

Commit message: Add files via upload
Parts:
- added R3, R7: 10k, Resistor_SMD:R_0603_1608Metric, symbol Device:R
Connections:
- net GND: now also R3.1
- net OUT: now also R3.2, R7.1; no longer ConnectionMain1.2 (Pin_2)
- new net: ConnectionMain1.2 (Pin_2), R7.2
Changed lines of the file:
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@@
   (junction (at 207.01 95.25) (diameter 0) (color 0 0 0 0)
+  )
+  (junction (at 106.68 25.4) (diameter 0) (color 0 0 0 0)
   )
   (junction (at 261.62 74.93) (diameter 0) (color 0 0 0 0)
@@
     (stroke (width 0) (type default) (color 0 0 0 0))
   )
+  (wire (pts (xy 106.68 41.91) (xy 113.03 41.91))
+    (stroke (width 0) (type default) (color 0 0 0 0))
+  )
   (wire (pts (xy 147.32 120.65) (xy 147.32 119.38))
     (stroke (width 0) (type default) (color 0 0 0 0))
@@
     (stroke (width 0) (type default) (color 0 0 0 0))
   )
+  (wire (pts (xy 106.68 25.4) (xy 106.68 41.91))
+    (stroke (width 0) (type default) (color 0 0 0 0))
+  )
   (wire (pts (xy 114.3 121.92) (xy 127 121.92))
     (stroke (width 0) (type default) (color 0 0 0 0))
@@
     (stroke (width 0) (type default) (color 0 0 0 0))
   )
+  (wire (pts (xy 113.03 41.91) (xy 113.03 64.77))
+    (stroke (width 0) (type default) (color 0 0 0 0))
+  )
   (wire (pts (xy 163.83 95.25) (xy 154.94 95.25))
     (stroke (width 0) (type default) (color 0 0 0 0))
@@
     (stroke (width 0) (type default) (color 0 0 0 0))
   )
+  (wire (pts (xy 106.68 25.4) (xy 110.49 25.4))
+    (stroke (width 0) (type default) (color 0 0 0 0))
+  )
   (wire (pts (xy 116.84 58.42) (xy 116.84 97.79))
     (stroke (width 0) (type default) (color 0 0 0 0))
@@
     (stroke (width 0) (type default) (color 0 0 0 0))
   )
+  (wire (pts (xy 102.87 25.4) (xy 106.68 25.4))
+    (stroke (width 0) (type default) (color 0 0 0 0))
+  )
   (wire (pts (xy 158.75 157.48) (xy 107.95 157.48))
     (stroke (width 0) (type default) (color 0 0 0 0))
@@
     (stroke (width 0) (type default) (color 0 0 0 0))
   )
-  (wire (pts (xy 118.11 25.4) (xy 118.11 64.77))
-    (stroke (width 0) (type default) (color 0 0 0 0))
-  )
   (wire (pts (xy 116.84 97.79) (xy 118.11 97.79))
     (stroke (width 0) (type default) (color 0 0 0 0))
@@
   )
   (wire (pts (xy 72.39 158.75) (xy 72.39 95.25))
+    (stroke (width 0) (type default) (color 0 0 0 0))
+  )
+  (wire (pts (xy 113.03 64.77) (xy 118.11 64.77))
     (stroke (width 0) (type default) (color 0 0 0 0))
   )
@@
   (text "Header - Tag Connect" (at 154.94 172.72 180)
     (effects (font (size 2.032 2.032)) (justify right bottom))
-  )
-  (label "OUT" (at 132.08 25.4 0)
-    (effects (font (size 1.27 1.27)) (justify left bottom))
   )
   (label "OUT" (at 118.11 64.77 90)
@@
     (pin "1")
   )
+  (symbol (lib_id "Device:R") (at 99.06 25.4 90) (unit 1)
+    (in_bom yes) (on_board yes)
+    (property "Reference" "R3" (id 0) (at 96.52 24.13 0)
+      (effects (font (size 1.27 1.27)) (justify left))
+    )
+    (property "Value" "10k" (id 1) (at 101.6 24.13 0)
+      (effects (font (size 1.27 1.27)) (justify left))
+    )
+    (property "Footprint" "Resistor_SMD:R_0603_1608Metric" (id 2) (at 99.06 27.178 90)
+      (effects (font (size 1.27 1.27)) hide)
+    )
+    (property "Datasheet" "~" (id 3) (at 99.06 25.4 0)
+      (effects (font (size 1.27 1.27)) hide)
+    )
+    (pin "1")
+    (pin "2")
+  )
   (symbol (lib_id "Device:C") (at 29.21 101.6 0) (unit 1)
     (in_bom yes) (on_board yes)
@@
     (pin "1")
     (pin "2")
+  )
+  (symbol (lib_id "power:GND") (at 95.25 25.4 270) (unit 1)
+    (in_bom yes) (on_board yes)
+    (property "Reference" "#PWR0103" (id 0) (at 88.9 25.4 0)
+      (effects (font (size 1.27 1.27)) hide)
+    )
+    (property "Value" "GND" (id 1) (at 90.17 25.4 0))
+    (property "Footprint" "" (id 2) (at 95.25 25.4 0)
+      (effects (font (size 1.27 1.27)) hide)
+    )
+    (property "Datasheet" "" (id 3) (at 95.25 25.4 0)
+      (effects (font (size 1.27 1.27)) hide)
+    )
+    (pin "1")
   )
   (symbol (lib_id "Device:C") (at 266.7 62.23 270) (unit 1)
@@
     (pin "1")
   )
+  (symbol (lib_id "Device:R") (at 114.3 25.4 90) (unit 1)
+    (in_bom yes) (on_board yes)
+    (property "Reference" "R7" (id 0) (at 111.76 24.13 0)
+      (effects (font (size 1.27 1.27)) (justify left))
+    )
+    (property "Value" "10k" (id 1) (at 116.84 24.13 0)
+      (effects (font (size 1.27 1.27)) (justify left))
+    )
+    (property "Footprint" "Resistor_SMD:R_0603_1608Metric" (id 2) (at 114.3 27.178 90)
+      (effects (font (size 1.27 1.27)) hide)
+    )
+    (property "Datasheet" "~" (id 3) (at 114.3 25.4 0)
+      (effects (font (size 1.27 1.27)) hide)
+    )
+    (pin "1")
+    (pin "2")
+  )
   (symbol (lib_id "power:GND") (at 273.05 158.75 0) (unit 1)
     (in_bom yes) (on_board yes) (fields_autoplaced)
@@
       (reference "#PWR0102") (unit 1) (value "GND") (footprint "")
     )
+    (path "/48edd299-f193-4939-b244-ac3e760e63bf"
+      (reference "#PWR0103") (unit 1) (value "GND") (footprint "")
+    )
     (path "/a2e977b9-6800-45b4-ae87-35d4429567ec"
       (reference "BT1") (unit 1) (value "3.6V") (footprint "Battery:BatteryHolder_Keystone_2460_1xAA")
@@
       (reference "R2") (unit 1) (value "10k") (footprint "Resistor_SMD:R_0603_1608Metric")
     )
+    (path "/3f22456a-f54e-4054-a9ca-35d4e5f21c04"
+      (reference "R3") (unit 1) (value "10k") (footprint "Resistor_SMD:R_0603_1608Metric")
+    )
     (path "/032c5c38-e792-4ad7-957d-8e019bf3c816"
       (reference "R4") (unit 1) (value "1M") (footprint "Resistor_SMD:R_0603_1608Metric")
@@
       (reference "R6") (unit 1) (value "100") (footprint "Resistor_SMD:R_0603_1608Metric")
     )
+    (path "/f7f2616c-5d66-4e7b-a13c-31aa295fe68d"
+      (reference "R7") (unit 1) (value "10k") (footprint "Resistor_SMD:R_0603_1608Metric")
+    )
     (path "/004b7c4b-8eee-4e9e-86f9-54258c6c8024"
